File: mFM-Rx/mFM-Rx.sch (KiCad schematic (older format))
At the start: 18 parts, among them P1 CONN_02X04, U1 nRF24L01+, Y1 16MHz, Y2 2450AT18A100E

Commit message: Updated schematics and PCBs
Other:
- note added: "1"
- moved on the sheet: U1
Changed lines of the file:
@@
 EESchema Schematic File Version 2
-LIBS:mFM-Rx-rescue
 LIBS:power
 LIBS:device
@@
 LIBS:atmel
 LIBS:contrib
-LIBS:nrf24l01+
 LIBS:valves
+LIBS:mFM_comp
 LIBS:mFM-Rx-cache
 EELAYER 25 0
@@
 encoding utf-8
 Sheet 1 1
-Title ""
-Date ""
-Rev ""
+Title "musicFromMotion Receiver"
+Date "2016-07-22"
+Rev "A"
 Comp ""
-Comment1 ""
-Comment2 ""
+Comment1 "By Calvin A. Cherry >> ccherry@riseup.net"
+Comment2 "Released under the TAPR Open Hardware License >> http://tapr.org/ohl.html"
 Comment3 ""
 Comment4 ""
@@
 L nRF24L01+ U1
 U 1 1 576F0F3B
-P 5100 2850
-F 0 "U1" H 4700 2450 60  0000 C CNN
-F 1 "nRF24L01+" H 4350 3250 60  0000 C CNN
-F 2 "mFM:QFN20_4x4" H 5100 2850 60  0001 C CNN
-F 3 "" H 5100 2850 60  0000 C CNN
-	1    5100 2850
+P 5100 2750
+F 0 "U1" H 4700 2250 60  0000 C CNN
+F 1 "nRF24L01+" H 4400 3100 60  0000 C CNN
+F 2 "mFM:QFN20_4x4" H 5100 2750 60  0001 C CNN
+F 3 "" H 5100 2750 60  0000 C CNN
+	1    5100 2750
 	1    0    0    -1
 $EndComp
@@
 	5100 3450 5750 3450
 Wire Wire Line
-	5750 4050 5750 2650
+	5750 2650 5750 4050
 Connection ~ 5100 3450
 Wire Wire Line
-	5200 4050 5750 4050
+	5750 4050 5250 4050
 Connection ~ 5750 3450
-Connection ~ 5300 4050
+Connection ~ 5050 3900
+Wire Wire Line
+	4750 2200 4750 2100
+Connection ~ 4750 2100
+Wire Wire Line
+	4450 2850 3600 2850
+Wire Wire Line
+	4900 3400 3100 3400
+Wire Wire Line
+	3100 3400 3100 2950
+Wire Wire Line
+	4450 2750 3750 2750
+Wire Wire Line
+	3750 2750 3750 2650
+Wire Wire Line
+	3750 2650 3600 2650
+Wire Wire Line
+	3600 2750 3700 2750
+Wire Wire Line
+	3700 2750 3700 2950
+Wire Wire Line
+	3700 2950 4450 2950
+Wire Wire Line
+	4450 2550 3100 2550
+Wire Wire Line
+	3100 2550 3100 2650
+Wire Wire Line
+	3800 2650 4450 2650
+Wire Wire Line
+	3800 2450 3800 2650
+Wire Wire Line
+	3800 2450 3000 2450
+Wire Wire Line
+	3000 2450 3000 2750
+Wire Wire Line
+	3000 2750 3100 2750
+Wire Wire Line
+	3100 2850 3000 2850
+Wire Wire Line
+	3000 2850 3000 2950
+Wire Wire Line
+	3600 2950 3650 2950
+Wire Wire Line
+	3650 2950 3650 2350
 $Comp
 L 2450AT18A100E Y2
-U 1 1 5770854B
+U 1 1 5792D858
 P 7500 2450
-F 0 "Y2" H 7600 2350 60  0000 C CNN
-F 1 "2450AT18A100E" H 7500 2850 60  0000 C CNN
+F 0 "Y2" H 7600 2300 60  0000 C CNN
+F 1 "2450AT18A100E" H 7500 2600 60  0000 C CNN
 F 2 "" H 7500 2450 60  0000 C CNN
 F 3 "" H 7500 2450 60  0000 C CNN
@@
 	1    0    0    -1
 $EndComp
-Connection ~ 5050 3900
-Wire Wire Line
-	4700 2200 4700 2100
-Connection ~ 4700 2100
-Wire Wire Line
-	4450 2850 3600 2850
-Wire Wire Line
-	4900 3400 3100 3400
-Wire Wire Line
-	3100 3400 3100 2950
-Wire Wire Line
-	4450 2750 3750 2750
-Wire Wire Line
-	3750 2750 3750 2650
-Wire Wire Line
-	3750 2650 3600 2650
-Wire Wire Line
-	3600 2750 3700 2750
-Wire Wire Line
-	3700 2750 3700 2950
-Wire Wire Line
-	3700 2950 4450 2950
-Wire Wire Line
-	4450 2550 3100 2550
-Wire Wire Line
-	3100 2550 3100 2650
-Wire Wire Line
-	3800 2650 4450 2650
-Wire Wire Line
-	3800 2450 3800 2650
-Wire Wire Line
-	3800 2450 3000 2450
-Wire Wire Line
-	3000 2450 3000 2750
-Wire Wire Line
-	3000 2750 3100 2750
-Wire Wire Line
-	3100 2850 3000 2850
-Wire Wire Line
-	3000 2850 3000 2950
-Wire Wire Line
-	3600 2950 3650 2950
-Wire Wire Line
-	3650 2950 3650 2350
+Text Notes 7280 7250 0    60   ~ 0
+1
+Text Notes 7380 7250 0    60   ~ 0
+1
 $EndSCHEMATC
