File: mFM-Tx/mFM-Tx.kicad_pcb (KiCad board)
At the start: 2 copper layers, 44 parts, among them P1 USB_micro, P2 CONN_01X05, SW1 SPDT, U1 MMA8653FCR1, U2 TC1015-2.8V, U3 AAT3681, U4 PIC16LF18323, U5 nRF24L01+, Y1 16MHz, Y2 2450AT18A100E

Commit message: Updated schematics and PCBs
Parts:
- added R11: R, Resistors_SMD:R_0402, F.Cu at (142.1, 109.7)
- added R12: R, Resistors_SMD:R_0402, F.Cu at (141.8, 108.0)
- added REF**: MountingHole_4mm, Mounting_Holes:MountingHole_4mm, F.Cu at (162.7, 99.5)
- added REF**: MountingHole_2.2mm_M2, Mounting_Holes:MountingHole_2.2mm_M2_DIN965, F.Cu at (163.4, 84.2)
- added REF**: MountingHole_2.2mm_M2, Mounting_Holes:MountingHole_2.2mm_M2_DIN965, F.Cu at (120.4, 84.1)
- added REF**: MountingHole_2.2mm_M2, Mounting_Holes:MountingHole_2.2mm_M2_DIN965, F.Cu at (120.4, 114.1)
- added REF**: MountingHole_4mm, Mounting_Holes:MountingHole_4mm, F.Cu at (121.2, 101.2)
- added REF**: MountingHole_2.2mm_M2, Mounting_Holes:MountingHole_2.2mm_M2_DIN965, F.Cu at (163.4, 114.1)
- moved Y2 61.1 mm to (119.8, 108.5), turned to 180 degrees
- moved C19 54.7 mm to (122.7, 107.3), turned to 270 degrees
- moved C18 54.5 mm to (123.3, 109.0), turned to 0 degrees
- moved L2 50.5 mm to (125.4, 109.0), turned to 180 degrees
- moved C16 49.2 mm to (125.2, 106.0), turned to 180 degrees
- moved L3 48.9 mm to (125.8, 107.4), turned to 90 degrees
- moved C14 47.6 mm to (129.1, 113.9), turned to 180 degrees
- moved L1 47.0 mm to (127.0, 108.5), turned to 90 degrees
- moved R10 46.9 mm to (128.8, 112.7), turned to 0 degrees
- moved C17 45.9 mm to (127.0, 106.5), turned to 90 degrees
- moved BT1 45.6 mm to (140.9, 93.8)
- moved C13 44.9 mm to (127.1, 104.1), turned to 90 degrees
- moved C15 43.6 mm to (131.4, 113.8), turned to 0 degrees
- moved C11 42.3 mm to (131.4, 112.6), turned to 0 degrees
- moved U5 41.4 mm to (130.3, 109.4), turned to 180 degrees
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Connections:
- D1 pad 1: /LED_K -> LED_K
- U3 pad 5: /LED_K -> LED_K
- U4 pad 4: Net-(U4-Pad4) -> /PIC_RD_NODENUM
- U4 pad 5: Net-(U4-Pad5) -> LED_K
Routing:
- net +BATT: track 17.2 -> 74.2 mm
- net GND: track 31.7 -> 84.2 mm, vias 0 -> 24
- net VDD: track 23.5 -> 68.8 mm, vias 0 -> 4
- net LED_K: track 0.00 -> 20.2 mm, vias 0 -> 2
- net ~IRQ: track 0.00 -> 7.53 mm
- net /CHGR_VBATT: track 14.7 -> 8.61 mm
- net MISO: track 0.00 -> 5.36 mm
- net MOSI: track 0.00 -> 4.79 mm, vias 0 -> 2
- net SCK: track 0.00 -> 4.45 mm
- net SCL: track 5.05 -> 9.34 mm
- net CE: track 0.00 -> 3.05 mm
- net /PIC_RD_NODENUM: track 0.00 -> 2.90 mm
- net ~CSN: track 0.00 -> 2.56 mm
- net SDA: track 5.35 -> 7.88 mm
- net /LED_K: track 2.30 -> 0.00 mm
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- added copper zone on B.Cu, net GND
- added copper zone on F.Cu, net GND
Other:
- board outline added: 50 x 37 mm
