File: mFM-Tx/mFM-Tx.kicad_pcb (KiCad board)
At the start: 2 copper layers, 50 x 37 mm, 53 parts, among them P1 USB_micro, P2 CONN_01X05, SW1 SPDT, U1 MMA8653FCR1, U2 TC1015-2.8V, U3 AAT3681, U4 PIC16LF18323, U5 nRF24L01+, Y1 16MHz, Y2 2450AT18A100E

Commit message: Created Tx gerbers
Parts:
- added BT1: Lipo battery, mFM:CR2450_clip, F.Cu at (176.4, 102.3)
- added BT1: Lipo battery, mFM:CR2450_clip, F.Cu at (176.4, 52.3)
- added BT1: Lipo battery, mFM:CR2450_clip, F.Cu at (127.7, 103.0)
- added BT1: Lipo battery, mFM:CR2450_clip, F.Cu at (75.7, 103.0)
- added BT1: Lipo battery, mFM:CR2450_clip, F.Cu at (127.7, 40.0)
- added C1: 0.1uF, Capacitors_SMD:C_0402, F.Cu at (191.4, 95.8)
- added C1: 0.1uF, Capacitors_SMD:C_0402, F.Cu at (191.4, 45.9)
- added C1: 0.1uF, Capacitors_SMD:C_0402, F.Cu at (134.1, 118.1)
- added C1: 0.1uF, Capacitors_SMD:C_0402, F.Cu at (82.1, 118.1)
- added C1: 0.1uF, Capacitors_SMD:C_0402, F.Cu at (134.1, 55.1)
- added C10: 0.1uF, Capacitors_SMD:C_0402, F.Cu at (196.0, 102.5)
- added C10: 0.1uF, Capacitors_SMD:C_0402, F.Cu at (196.0, 52.5)
- added C10: 0.1uF, Capacitors_SMD:C_0402, F.Cu at (127.4, 122.7)
- added C10: 0.1uF, Capacitors_SMD:C_0402, F.Cu at (75.4, 122.7)
- added C10: 0.1uF, Capacitors_SMD:C_0402, F.Cu at (127.4, 59.6)
- added C11: 33nF, Capacitors_SMD:C_0402, F.Cu at (195.6, 112.8)
- added C11: 33nF, Capacitors_SMD:C_0402, F.Cu at (195.6, 62.8)
- added C11: 33nF, Capacitors_SMD:C_0402, F.Cu at (117.1, 122.3)
- added C11: 33nF, Capacitors_SMD:C_0402, F.Cu at (65.1, 122.3)
- added C11: 33nF, Capacitors_SMD:C_0402, F.Cu at (117.1, 59.3)
- added C12: 22pF, Capacitors_SMD:C_0402, F.Cu at (185.8, 114.7)
- added C12: 22pF, Capacitors_SMD:C_0402, F.Cu at (185.8, 64.7)
- added C12: 22pF, Capacitors_SMD:C_0402, F.Cu at (115.3, 112.4)
- added C12: 22pF, Capacitors_SMD:C_0402, F.Cu at (63.3, 112.4)
- added C12: 22pF, Capacitors_SMD:C_0402, F.Cu at (115.3, 49.4)
- added C13: 22pF, Capacitors_SMD:C_0402, F.Cu at (187.1, 117.1)
- added C13: 22pF, Capacitors_SMD:C_0402, F.Cu at (187.1, 67.1)
- added C13: 22pF, Capacitors_SMD:C_0402, F.Cu at (112.8, 113.8)
- added C13: 22pF, Capacitors_SMD:C_0402, F.Cu at (60.8, 113.8)
- added C13: 22pF, Capacitors_SMD:C_0402, F.Cu at (112.8, 50.8)
- added C14: 10nF, Capacitors_SMD:C_0402, F.Cu at (196.9, 115.1)
- added C14: 10nF, Capacitors_SMD:C_0402, F.Cu at (196.9, 65.1)
- added C14: 10nF, Capacitors_SMD:C_0402, F.Cu at (114.8, 123.6)
- added C14: 10nF, Capacitors_SMD:C_0402, F.Cu at (62.8, 123.6)
- added C14: 10nF, Capacitors_SMD:C_0402, F.Cu at (114.8, 60.6)
- added C15: 1nF, Capacitors_SMD:C_0402, F.Cu at (196.8, 112.8)
- added C15: 1nF, Capacitors_SMD:C_0402, F.Cu at (196.8, 62.8)
- added C15: 1nF, Capacitors_SMD:C_0402, F.Cu at (117.1, 123.5)
- added C15: 1nF, Capacitors_SMD:C_0402, F.Cu at (65.1, 123.5)
- added C15: 1nF, Capacitors_SMD:C_0402, F.Cu at (117.1, 60.5)
- added C16: 2.2nF, Capacitors_SMD:C_0402, F.Cu at (189.1, 119.0)
- added C16: 2.2nF, Capacitors_SMD:C_0402, F.Cu at (189.1, 69.0)
- added C16: 2.2nF, Capacitors_SMD:C_0402, F.Cu at (111.0, 115.7)
- added C16: 2.2nF, Capacitors_SMD:C_0402, F.Cu at (59.0, 115.7)
- added C16: 2.2nF, Capacitors_SMD:C_0402, F.Cu at (111.0, 52.7)
- added C17: 4.7pF, Capacitors_SMD:C_0402, F.Cu at (189.4, 117.2)
- added C17: 4.7pF, Capacitors_SMD:C_0402, F.Cu at (189.4, 67.2)
- added C17: 4.7pF, Capacitors_SMD:C_0402, F.Cu at (112.7, 116.1)
- added C17: 4.7pF, Capacitors_SMD:C_0402, F.Cu at (60.7, 116.1)
- added C17: 4.7pF, Capacitors_SMD:C_0402, F.Cu at (112.7, 53.1)
- added C18: 1.5pF, Capacitors_SMD:C_0402, F.Cu at (192.0, 121.0)
- added C18: 1.5pF, Capacitors_SMD:C_0402, F.Cu at (192.0, 71.0)
- added C18: 1.5pF, Capacitors_SMD:C_0402, F.Cu at (109.0, 118.7)
- added C18: 1.5pF, Capacitors_SMD:C_0402, F.Cu at (57.0, 118.7)
- added C18: 1.5pF, Capacitors_SMD:C_0402, F.Cu at (109.0, 55.7)
- added C19: 1pF, Capacitors_SMD:C_0402, F.Cu at (190.3, 121.5)
- added C19: 1pF, Capacitors_SMD:C_0402, F.Cu at (190.3, 71.5)
- added C19: 1pF, Capacitors_SMD:C_0402, F.Cu at (108.4, 116.9)
- added C19: 1pF, Capacitors_SMD:C_0402, F.Cu at (56.4, 116.9)
- added C19: 1pF, Capacitors_SMD:C_0402, F.Cu at (108.4, 53.9)
- added C2: 1uF, Capacitors_SMD:C_0402, F.Cu at (194.3, 100.3)
- added C2: 1uF, Capacitors_SMD:C_0402, F.Cu at (194.3, 50.3)
- added C2: 1uF, Capacitors_SMD:C_0402, F.Cu at (129.7, 121.0)
- added C2: 1uF, Capacitors_SMD:C_0402, F.Cu at (77.7, 121.0)
- added C2: 1uF, Capacitors_SMD:C_0402, F.Cu at (129.7, 58.0)
- added C3: 0.1uF, Capacitors_SMD:C_0402, F.Cu at (195.7, 95.9)
- added C3: 0.1uF, Capacitors_SMD:C_0402, F.Cu at (195.7, 45.9)
- added C3: 0.1uF, Capacitors_SMD:C_0402, F.Cu at (134.0, 122.4)
- added C3: 0.1uF, Capacitors_SMD:C_0402, F.Cu at (82.0, 122.4)
- added C3: 0.1uF, Capacitors_SMD:C_0402, F.Cu at (134.0, 59.4)
- added C4: 10uF, Capacitors_SMD:C_0805, F.Cu at (189.9, 86.6)
- added C4: 10uF, Capacitors_SMD:C_0805, F.Cu at (189.9, 36.6)
- added C4: 10uF, Capacitors_SMD:C_0805, F.Cu at (143.3, 116.6)
- added C4: 10uF, Capacitors_SMD:C_0805, F.Cu at (91.3, 116.6)
- added C4: 10uF, Capacitors_SMD:C_0805, F.Cu at (143.3, 53.6)
- added C5: 1uF, Capacitors_SMD:C_0402, F.Cu at (193.1, 92.6)
- added C5: 1uF, Capacitors_SMD:C_0402, F.Cu at (193.1, 42.6)
- added C5: 1uF, Capacitors_SMD:C_0402, F.Cu at (137.3, 119.8)
- added C5: 1uF, Capacitors_SMD:C_0402, F.Cu at (85.3, 119.8)
- added C5: 1uF, Capacitors_SMD:C_0402, F.Cu at (137.3, 56.8)
- added C6: 1uF, Capacitors_SMD:C_0402, F.Cu at (193.1, 87.3)
- added C6: 1uF, Capacitors_SMD:C_0402, F.Cu at (193.1, 37.4)
- added C6: 1uF, Capacitors_SMD:C_0402, F.Cu at (142.6, 119.8)
- added C6: 1uF, Capacitors_SMD:C_0402, F.Cu at (90.6, 119.8)
- added C6: 1uF, Capacitors_SMD:C_0402, F.Cu at (142.6, 56.8)
- added C7: 0.1uF, Capacitors_SMD:C_0402, F.Cu at (193.9, 99.1)
- added C7: 0.1uF, Capacitors_SMD:C_0402, F.Cu at (193.9, 49.1)
- added C7: 0.1uF, Capacitors_SMD:C_0402, F.Cu at (130.9, 120.6)
- added C7: 0.1uF, Capacitors_SMD:C_0402, F.Cu at (78.9, 120.6)
- added C7: 0.1uF, Capacitors_SMD:C_0402, F.Cu at (130.9, 57.6)
- added C8: 470pF, Capacitors_SMD:C_0402, F.Cu at (187.8, 91.4)
- added C8: 470pF, Capacitors_SMD:C_0402, F.Cu at (187.8, 41.4)
- added C8: 470pF, Capacitors_SMD:C_0402, F.Cu at (138.6, 114.4)
- added C8: 470pF, Capacitors_SMD:C_0402, F.Cu at (86.5, 114.4)
- added C8: 470pF, Capacitors_SMD:C_0402, F.Cu at (138.6, 51.4)
- added C9: 1uF, Capacitors_SMD:C_0402, F.Cu at (188.3, 93.2)
- added C9: 1uF, Capacitors_SMD:C_0402, F.Cu at (188.3, 43.1)
- added C9: 1uF, Capacitors_SMD:C_0402, F.Cu at (136.8, 115.0)
- added C9: 1uF, Capacitors_SMD:C_0402, F.Cu at (84.8, 115.0)
- added C9: 1uF, Capacitors_SMD:C_0402, F.Cu at (136.8, 52.0)
- added D1: LED, LEDs:LED_0402, F.Cu at (187.2, 88.0)
- added D1: LED, LEDs:LED_0402, F.Cu at (187.2, 38.0)
- added D1: LED, LEDs:LED_0402, F.Cu at (142.0, 113.8)
- added D1: LED, LEDs:LED_0402, F.Cu at (90.0, 113.8)
- added D1: LED, LEDs:LED_0402, F.Cu at (142.0, 50.9)
- added L1: 8.2nH, Resistors_SMD:R_0402, F.Cu at (191.6, 117.2)
- added L1: 8.2nH, Resistors_SMD:R_0402, F.Cu at (191.6, 67.2)
- added L1: 8.2nH, Resistors_SMD:R_0402, F.Cu at (112.7, 118.2)
- added L1: 8.2nH, Resistors_SMD:R_0402, F.Cu at (60.7, 118.2)
- added L1: 8.2nH, Resistors_SMD:R_0402, F.Cu at (112.7, 55.2)
- added L2: 3.9nH, Resistors_SMD:R_0402, F.Cu at (192.0, 118.8)
- added L2: 3.9nH, Resistors_SMD:R_0402, F.Cu at (192.0, 68.8)
- added L2: 3.9nH, Resistors_SMD:R_0402, F.Cu at (111.1, 118.7)
- added L2: 3.9nH, Resistors_SMD:R_0402, F.Cu at (59.1, 118.7)
- added L2: 3.9nH, Resistors_SMD:R_0402, F.Cu at (111.1, 55.6)
- added L3: 2.7nH, Resistors_SMD:R_0402, F.Cu at (190.4, 118.5)
- added L3: 2.7nH, Resistors_SMD:R_0402, F.Cu at (190.4, 68.5)
- added L3: 2.7nH, Resistors_SMD:R_0402, F.Cu at (111.5, 117.0)
- added L3: 2.7nH, Resistors_SMD:R_0402, F.Cu at (59.5, 117.0)
- added L3: 2.7nH, Resistors_SMD:R_0402, F.Cu at (111.5, 54.0)
- added P1: USB_micro, Connect:USB_Micro-B_10103594-0001LF, F.Cu at (191.0, 82.0)
- added P1: USB_micro, Connect:USB_Micro-B_10103594-0001LF, F.Cu at (191.0, 32.0)
- added P1: USB_micro, Connect:USB_Micro-B_10103594-0001LF, F.Cu at (147.9, 117.7)
- added P1: USB_micro, Connect:USB_Micro-B_10103594-0001LF, F.Cu at (96.0, 117.7)
- added P1: USB_micro, Connect:USB_Micro-B_10103594-0001LF, F.Cu at (147.9, 54.6)
- added P2: CONN_01X05, Socket_Strips:Socket_Strip_Straight_1x05, F.Cu at (198.9, 100.2)
- added P2: CONN_01X05, Socket_Strips:Socket_Strip_Straight_1x05, F.Cu at (198.9, 50.2)
- added P2: CONN_01X05, Socket_Strips:Socket_Strip_Straight_1x05, F.Cu at (129.8, 125.5)
- added P2: CONN_01X05, Socket_Strips:Socket_Strip_Straight_1x05, F.Cu at (77.8, 125.5)
- added P2: CONN_01X05, Socket_Strips:Socket_Strip_Straight_1x05, F.Cu at (129.8, 62.5)
- added R1: 1k, Resistors_SMD:R_0402, F.Cu at (195.8, 98.4)
- added R1: 1k, Resistors_SMD:R_0402, F.Cu at (195.8, 48.4)
- added R1: 1k, Resistors_SMD:R_0402, F.Cu at (131.6, 122.4)
- added R1: 1k, Resistors_SMD:R_0402, F.Cu at (79.6, 122.4)
- added R1: 1k, Resistors_SMD:R_0402, F.Cu at (131.6, 59.4)
- added R10: 22k, Resistors_SMD:R_0402, F.Cu at (195.7, 115.4)
- added R10: 22k, Resistors_SMD:R_0402, F.Cu at (195.7, 65.4)
- added R10: 22k, Resistors_SMD:R_0402, F.Cu at (114.5, 122.3)
- added R10: 22k, Resistors_SMD:R_0402, F.Cu at (62.5, 122.3)
- added R10: 22k, Resistors_SMD:R_0402, F.Cu at (114.5, 59.3)
- added R11: R, Resistors_SMD:R_0402, F.Cu at (192.7, 102.2)
- added R11: R, Resistors_SMD:R_0402, F.Cu at (192.7, 52.2)
- added R11: R, Resistors_SMD:R_0402, F.Cu at (127.8, 119.3)
- added R11: R, Resistors_SMD:R_0402, F.Cu at (75.8, 119.3)
- added R11: R, Resistors_SMD:R_0402, F.Cu at (127.8, 56.3)
- added R12: R, Resistors_SMD:R_0402, F.Cu at (191.1, 102.5)
- added R12: R, Resistors_SMD:R_0402, F.Cu at (191.1, 52.5)
- added R12: R, Resistors_SMD:R_0402, F.Cu at (127.5, 117.7)
- added R12: R, Resistors_SMD:R_0402, F.Cu at (75.5, 117.7)
- added R12: R, Resistors_SMD:R_0402, F.Cu at (127.5, 54.7)
- added R2: 16.2k, Resistors_SMD:R_0402, F.Cu at (193.2, 89.8)
- added R2: 16.2k, Resistors_SMD:R_0402, F.Cu at (193.2, 39.8)
- added R2: 16.2k, Resistors_SMD:R_0402, F.Cu at (140.2, 119.8)
- added R2: 16.2k, Resistors_SMD:R_0402, F.Cu at (88.2, 119.8)
- added R2: 16.2k, Resistors_SMD:R_0402, F.Cu at (140.2, 56.8)
- added R3: 1k, Resistors_SMD:R_0402, F.Cu at (191.4, 98.7)
- added R3: 1k, Resistors_SMD:R_0402, F.Cu at (191.4, 48.7)
- added R3: 1k, Resistors_SMD:R_0402, F.Cu at (131.2, 118.0)
- added R3: 1k, Resistors_SMD:R_0402, F.Cu at (79.2, 118.0)
- added R3: 1k, Resistors_SMD:R_0402, F.Cu at (131.2, 55.0)
- added R4: 1k, Resistors_SMD:R_0402, F.Cu at (185.3, 88.0)
- added R4: 1k, Resistors_SMD:R_0402, F.Cu at (185.3, 38.0)
- added R4: 1k, Resistors_SMD:R_0402, F.Cu at (142.0, 112.0)
- added R4: 1k, Resistors_SMD:R_0402, F.Cu at (90.0, 112.0)
- added R4: 1k, Resistors_SMD:R_0402, F.Cu at (142.0, 49.0)
- added R5: 10k, Resistors_SMD:R_0402, F.Cu at (196.4, 101.3)
- added R5: 10k, Resistors_SMD:R_0402, F.Cu at (196.4, 51.3)
- added R5: 10k, Resistors_SMD:R_0402, F.Cu at (128.7, 123.1)
- added R5: 10k, Resistors_SMD:R_0402, F.Cu at (76.7, 123.1)
- added R5: 10k, Resistors_SMD:R_0402, F.Cu at (128.7, 60.1)
- added R6: 46.5k, Resistors_SMD:R_0402, F.Cu at (190.5, 104.6)
- added R6: 46.5k, Resistors_SMD:R_0402, F.Cu at (190.5, 54.6)
- added R6: 46.5k, Resistors_SMD:R_0402, F.Cu at (125.3, 117.2)
- added R6: 46.5k, Resistors_SMD:R_0402, F.Cu at (73.3, 117.2)
- added R6: 46.5k, Resistors_SMD:R_0402, F.Cu at (125.3, 54.1)
- added R7: 100k, Resistors_SMD:R_0402, F.Cu at (190.5, 106.5)
- added R7: 100k, Resistors_SMD:R_0402, F.Cu at (190.5, 56.5)
- added R7: 100k, Resistors_SMD:R_0402, F.Cu at (123.5, 117.2)
- added R7: 100k, Resistors_SMD:R_0402, F.Cu at (71.5, 117.2)
- added R7: 100k, Resistors_SMD:R_0402, F.Cu at (123.5, 54.1)
- added R8: 0, Resistors_SMD:R_0402, F.Cu at (195.3, 109.4)
- added R8: 0, Resistors_SMD:R_0402, F.Cu at (195.3, 59.4)
- added R8: 0, Resistors_SMD:R_0402, F.Cu at (120.5, 122.0)
- added R8: 0, Resistors_SMD:R_0402, F.Cu at (68.5, 122.0)
- added R8: 0, Resistors_SMD:R_0402, F.Cu at (120.5, 59.0)
- added R9: 0, Resistors_SMD:R_0402, F.Cu at (194.0, 109.4)
- added R9: 0, Resistors_SMD:R_0402, F.Cu at (194.0, 59.4)
- added R9: 0, Resistors_SMD:R_0402, F.Cu at (120.5, 120.7)
- added R9: 0, Resistors_SMD:R_0402, F.Cu at (68.5, 120.7)
- added R9: 0, Resistors_SMD:R_0402, F.Cu at (120.5, 57.7)
- added REF**: Symbol_OSHW-Logo_CopperTop_Negative, Symbols:Symbol_OSHW-Logo_CopperTop_Negative, F.Cu at (167.1, 102.3)
- added REF**: MountingHole_2.2mm_M2, Mounting_Holes:MountingHole_2.2mm_M2_DIN965, F.Cu at (167.1, 73.8)
- added REF**: MountingHole_2.2mm_M2, Mounting_Holes:MountingHole_2.2mm_M2_DIN965, F.Cu at (197.1, 73.8)
- added REF**: MountingHole_4mm, Mounting_Holes:MountingHole_4mm, F.Cu at (183.6, 73.0)
- added REF**: MountingHole_2.2mm_M2, Mounting_Holes:MountingHole_2.2mm_M2_DIN965, F.Cu at (197.1, 30.9)
- added REF**: Symbol_OSHW-Logo_CopperTop_Negative, Symbols:Symbol_OSHW-Logo_CopperTop_Negative, F.Cu at (167.1, 52.3)
- added REF**: Symbol_OSHW-Logo_CopperTop_Negative, Symbols:Symbol_OSHW-Logo_CopperTop_Negative, F.Cu at (127.7, 93.7)
- added REF**: MountingHole_2.2mm_M2, Mounting_Holes:MountingHole_2.2mm_M2_DIN965, F.Cu at (149.1, 123.8)
- added REF**: MountingHole_4mm, Mounting_Holes:MountingHole_4mm, F.Cu at (106.9, 110.2)
- added REF**: MountingHole_2.2mm_M2, Mounting_Holes:MountingHole_2.2mm_M2_DIN965, F.Cu at (106.1, 123.8)
- added REF**: MountingHole_2.2mm_M2, Mounting_Holes:MountingHole_2.2mm_M2_DIN965, F.Cu at (106.1, 93.8)
- added REF**: MountingHole_2.2mm_M2, Mounting_Holes:MountingHole_2.2mm_M2_DIN965, F.Cu at (197.1, 80.8)
- added REF**: MountingHole_2.2mm_M2, Mounting_Holes:MountingHole_2.2mm_M2_DIN965, F.Cu at (149.2, 93.8)
- added REF**: MountingHole_4mm, Mounting_Holes:MountingHole_4mm, F.Cu at (148.4, 109.2)
- added REF**: MountingHole_4mm, Mounting_Holes:MountingHole_4mm, F.Cu at (96.4, 109.2)
- added REF**: MountingHole_2.2mm_M2, Mounting_Holes:MountingHole_2.2mm_M2_DIN965, F.Cu at (97.2, 93.8)
- added REF**: MountingHole_2.2mm_M2, Mounting_Holes:MountingHole_2.2mm_M2_DIN965, F.Cu at (54.1, 93.8)
- added REF**: MountingHole_2.2mm_M2, Mounting_Holes:MountingHole_2.2mm_M2_DIN965, F.Cu at (54.1, 123.8)
- added REF**: MountingHole_4mm, Mounting_Holes:MountingHole_4mm, F.Cu at (54.9, 110.2)
- added REF**: MountingHole_2.2mm_M2, Mounting_Holes:MountingHole_2.2mm_M2_DIN965, F.Cu at (97.1, 123.8)
- added REF**: Symbol_OSHW-Logo_CopperTop_Negative, Symbols:Symbol_OSHW-Logo_CopperTop_Negative, F.Cu at (75.7, 93.7)
- added REF**: Symbol_OSHW-Logo_CopperTop_Negative, Symbols:Symbol_OSHW-Logo_CopperTop_Negative, F.Cu at (127.7, 30.7)
- added REF**: MountingHole_4mm, Mounting_Holes:MountingHole_4mm, F.Cu at (183.6, 123.0)
- added REF**: MountingHole_2.2mm_M2, Mounting_Holes:MountingHole_2.2mm_M2_DIN965, F.Cu at (149.1, 60.8)
- added REF**: MountingHole_4mm, Mounting_Holes:MountingHole_4mm, F.Cu at (106.9, 47.2)
- added REF**: MountingHole_2.2mm_M2, Mounting_Holes:MountingHole_2.2mm_M2_DIN965, F.Cu at (106.1, 60.8)
- added REF**: MountingHole_2.2mm_M2, Mounting_Holes:MountingHole_2.2mm_M2_DIN965, F.Cu at (106.1, 30.8)
- added REF**: MountingHole_2.2mm_M2, Mounting_Holes:MountingHole_2.2mm_M2_DIN965, F.Cu at (149.2, 30.8)
- added REF**: MountingHole_4mm, Mounting_Holes:MountingHole_4mm, F.Cu at (148.4, 46.2)
- added REF**: MountingHole_2.2mm_M2, Mounting_Holes:MountingHole_2.2mm_M2_DIN965, F.Cu at (197.1, 123.8)
- added REF**: MountingHole_2.2mm_M2, Mounting_Holes:MountingHole_2.2mm_M2_DIN965, F.Cu at (167.1, 123.8)
- added REF**: MountingHole_2.2mm_M2, Mounting_Holes:MountingHole_2.2mm_M2_DIN965, F.Cu at (167.2, 80.8)
- added REF**: MountingHole_4mm, Mounting_Holes:MountingHole_4mm, F.Cu at (182.6, 81.5)
- added REF**: MountingHole_4mm, Mounting_Holes:MountingHole_4mm, F.Cu at (182.6, 31.6)
- added REF**: MountingHole_2.2mm_M2, Mounting_Holes:MountingHole_2.2mm_M2_DIN965, F.Cu at (167.2, 30.8)
- added SW1: SPDT, mFM:SW_SPDT_SMD, F.Cu at (197.0, 89.7)
- added SW1: SPDT, mFM:SW_SPDT_SMD, F.Cu at (197.0, 39.7)
- added SW1: SPDT, mFM:SW_SPDT_SMD, F.Cu at (140.2, 123.7)
- added SW1: SPDT, mFM:SW_SPDT_SMD, F.Cu at (88.2, 123.7)
- added SW1: SPDT, mFM:SW_SPDT_SMD, F.Cu at (140.2, 60.6)
- added U1: MMA8653FCR1, mFM:DFN-10-2mmx2mm, F.Cu at (193.6, 97.0)
- added U1: MMA8653FCR1, mFM:DFN-10-2mmx2mm, F.Cu at (193.6, 47.0)
- added U1: MMA8653FCR1, mFM:DFN-10-2mmx2mm, F.Cu at (133.0, 120.2)
- added U1: MMA8653FCR1, mFM:DFN-10-2mmx2mm, F.Cu at (81.0, 120.2)
- added U1: MMA8653FCR1, mFM:DFN-10-2mmx2mm, F.Cu at (133.0, 57.2)
- added U2: TC1015-2.8V, TO_SOT_Packages_SMD:SOT-23-5, F.Cu at (190.8, 92.8)
- added U2: TC1015-2.8V, TO_SOT_Packages_SMD:SOT-23-5, F.Cu at (190.8, 42.8)
- added U2: TC1015-2.8V, TO_SOT_Packages_SMD:SOT-23-5, F.Cu at (137.2, 117.5)
- added U2: TC1015-2.8V, TO_SOT_Packages_SMD:SOT-23-5, F.Cu at (85.2, 117.5)
- added U2: TC1015-2.8V, TO_SOT_Packages_SMD:SOT-23-5, F.Cu at (137.2, 54.5)
- added U3: AAT3681, mFM:SC70JW-8, F.Cu at (190.8, 88.8)
- added U3: AAT3681, mFM:SC70JW-8, F.Cu at (190.8, 38.8)
- added U3: AAT3681, mFM:SC70JW-8, F.Cu at (141.2, 117.5)
- added U3: AAT3681, mFM:SC70JW-8, F.Cu at (89.2, 117.5)
- added U3: AAT3681, mFM:SC70JW-8, F.Cu at (141.2, 54.5)
- added U4: PIC16LF18323, mFM:UQFN-16_4x4mm_Pitch0.65mm_Pad2x2mm, F.Cu at (193.8, 105.8)
- added U4: PIC16LF18323, mFM:UQFN-16_4x4mm_Pitch0.65mm_Pad2x2mm, F.Cu at (193.8, 55.8)
- added U4: PIC16LF18323, mFM:UQFN-16_4x4mm_Pitch0.65mm_Pad2x2mm, F.Cu at (124.1, 120.5)
- added U4: PIC16LF18323, mFM:UQFN-16_4x4mm_Pitch0.65mm_Pad2x2mm, F.Cu at (72.1, 120.5)
- added U4: PIC16LF18323, mFM:UQFN-16_4x4mm_Pitch0.65mm_Pad2x2mm, F.Cu at (124.1, 57.5)
- added U5: nRF24L01+, mFM:VFQFN-20_4x4mm_Pitch0.5mm_Pad2x2mm, F.Cu at (192.4, 114.0)
- added U5: nRF24L01+, mFM:VFQFN-20_4x4mm_Pitch0.5mm_Pad2x2mm, F.Cu at (192.4, 64.0)
- added U5: nRF24L01+, mFM:VFQFN-20_4x4mm_Pitch0.5mm_Pad2x2mm, F.Cu at (116.0, 119.0)
- added U5: nRF24L01+, mFM:VFQFN-20_4x4mm_Pitch0.5mm_Pad2x2mm, F.Cu at (64.0, 119.0)
- added U5: nRF24L01+, mFM:VFQFN-20_4x4mm_Pitch0.5mm_Pad2x2mm, F.Cu at (116.0, 56.0)
- added Y1: 16MHz, mFM:ABM8, F.Cu at (188.0, 114.5)
- added Y1: 16MHz, mFM:ABM8, F.Cu at (188.0, 64.5)
- added Y1: 16MHz, mFM:ABM8, F.Cu at (115.5, 114.7)
- added Y1: 16MHz, mFM:ABM8, F.Cu at (63.5, 114.7)
- added Y1: 16MHz, mFM:ABM8, F.Cu at (115.5, 51.7)
- added Y2: 2450AT18A100E, mFM:2450AT, F.Cu at (191.6, 124.5)
- added Y2: 2450AT18A100E, mFM:2450AT, F.Cu at (191.6, 74.5)
- added Y2: 2450AT18A100E, mFM:2450AT, F.Cu at (105.5, 118.2)
- added Y2: 2450AT18A100E, mFM:2450AT, F.Cu at (53.5, 118.2)
- added Y2: 2450AT18A100E, mFM:2450AT, F.Cu at (105.5, 55.2)
- moved C1 85.1 mm to (82.1, 55.1)
- moved C11 85.1 mm to (65.1, 59.3)
- moved C15 85.1 mm to (65.1, 60.5)
- moved C18 85.1 mm to (57.0, 55.7)
- moved C4 85.1 mm to (91.3, 53.6)
- moved D1 85.1 mm to (90.0, 50.9)
- moved L2 85.1 mm to (59.1, 55.6)
- moved R11 85.1 mm to (75.8, 56.3)
- moved R3 85.1 mm to (79.2, 55.0)
- moved R6 85.1 mm to (73.3, 54.1)
- moved SW1 85.1 mm to (88.2, 60.6)
- moved U4 85.1 mm to (72.1, 57.5)
- moved U5 85.1 mm to (64.0, 56.0)
- moved Y1 85.1 mm to (63.5, 51.7)
- moved BT1 85.1 mm to (75.7, 40.0)
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Routing:
- net GND: track 89.1 -> 534.4 mm, vias 28 -> 168
- net +BATT: track 75.5 -> 453.0 mm
- net VDD: track 68.8 -> 413.0 mm, vias 4 -> 24
- net LED_K: track 20.2 -> 121.3 mm, vias 2 -> 12
- net /LDO_VBATT: track 13.1 -> 78.4 mm
- net SCL: track 9.34 -> 56.0 mm
- net /CHGR_VBATT: track 8.61 -> 51.7 mm
- net /VUSB: track 8.31 -> 49.8 mm
- net VPP: track 8.08 -> 48.5 mm, vias 2 -> 12
- net SDA: track 7.88 -> 47.3 mm
- net ~IRQ: track 7.53 -> 45.2 mm
- net ICSPCLK: track 7.01 -> 42.0 mm
- net ICSPDAT: track 5.48 -> 32.9 mm
- net /NRF_XC2: track 5.42 -> 32.5 mm
- net MISO: track 5.36 -> 32.2 mm
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Other:
- board size 50 x 37 mm -> 150 x 100 mm
- board text added: "^ v-cut ^"
- board text added: "mFM-Tx Rv.A"
- board text added: "v-cut ->"
- board text removed: "mFM-Tx R1.0"
