File: mFM-Tx/mFM-Tx.sch (KiCad schematic (older format))
At the start: 44 parts, among them P1 USB_micro, P2 CONN_01X05, SW1 SPDT, U1 MMA8653FCR1, U2 TC1015-2.8V, U3 AAT3681, U4 PIC16LF18323, U5 nRF24L01+, Y1 16MHz, Y2 2450AT18A100E

Commit message: Updated schematics and PCBs
Parts:
- added R11, R12: R, Resistors_SMD:R_0402, symbol R
Connections:
- net GND: now also R12.1
- net LED_K: now also U4.5 (RC4)
- net VDD: now also R11.2
- net PIC_RD_NODENUM: now reaches U4.4 (RC5)
- net PIC_RD_NODENUM: now also R11.1, R12.2
- no-connect marks 9 -> 7
Other:
- note added: "1"

Commit message: Created Tx gerbers
Other:
- note removed: "1"
Changed lines of the file:
@@
 encoding utf-8
 Sheet 1 1
-Title "musicFromMotion"
+Title "musicFromMotion Transmitter (Tx)"
 Date "2016-07-22"
 Rev "A"
@@
 	1    0    0    -1
 $EndComp
-Text Notes 7280 7250 0    60   ~ 0
-1
-Text Notes 7380 7250 0    60   ~ 0
-1
 $Comp
 L R R11
