File: hardware/mFM-Tx_0.1/mFM-Tx_0.1.kicad_pcb (KiCad board)
At the start: 2 copper layers, 38 x 51.6 mm, 28 parts, among them P1 Header_1x6, P2 Header_1x9, P3 Header_2x3, P4 Header_1x5, P5 Header_1x2, P6 Header_1x2, Q1 ATmega368P-AU, SW1 SPDT, U1 TC1015-2.8V

Commit message: Updated gerbers for Tx_0.1 and _0.2
Other:
- board text removed: "TODO: - Label switch states (ON or OFF/CHARGE)"
Changed lines of the file:
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@@
     (area 128.919048 76.225 189.102953 149.125)
     (thickness 1.6)
-    (drawings 60)
+    (drawings 59)
     (tracks 261)
     (zones 0)
@@
     (visible_elements FFFFFF7F)
     (pcbplotparams
-      (layerselection 0x01030_80000001)
+      (layerselection 0x010f0_80000001)
       (usegerberextensions true)
       (excludeedgelayer true)
@@
     (effects (font (size 0.8 0.8) (thickness 0.15)) (justify left mirror))
   )
-  (gr_text "TODO:\n- Label switch states (ON or OFF/CHARGE)" (at 137 78.7) (layer B.Fab)
-    (effects (font (size 1.5 1.5) (thickness 0.3)) (justify left))
-  )
   (gr_text GND (at 153 100.2 90) (layer B.SilkS)
